File: PCBs/Lab4/Lab4.kicad_pcb (KiCad board)
At the start: 2 copper layers, 13 parts, among them IC1 M0C1103QDDFRQ1, J1 Conn_01x05_Pin, SW1 SW_SPST, SW2 SW_SPST

Commit message: lab4 completed
Parts:
- removed D3: NeoPixel_THT, LED_THT:LED_D5.0mm-4_RGB_Staggered_Pins
- removed SW1: SW_SPST, Button_Switch_THT:SW_PUSH_6mm_H5mm
- BT1, C1, C2, C3, R1, R2, SW2: moved to B.Cu
- moved SW2 37.2 mm to (125.5, 120.5), turned to 180 degrees
- moved R1 29.7 mm to (126.5, 111.0), turned to 90 degrees
- moved R2 27.6 mm to (129.0, 115.0), turned to 180 degrees
- moved C1 25.1 mm to (131.5, 120.0), turned to -90 degrees
- moved C3 22.6 mm to (127.0, 102.6), turned to 90 degrees
- moved TH1 21.9 mm to (136.6, 120.5), turned to 180 degrees
- moved J1 20.5 mm to (123.0, 102.4)
- moved C2 15.6 mm to (144.0, 120.0), turned to -90 degrees
- moved BT1 14.9 mm to (136.6, 107.3)
- moved IC1 12.0 mm to (136.6, 114.5), turned to 180 degrees
- moved D2 5.15 mm to (136.6, 107.2)
Routing:
- net VDD: track 0.00 -> 100.0 mm, vias 0 -> 2
- net THRM: track 0.00 -> 30.7 mm, vias 0 -> 1
- net NRST: track 0.00 -> 29.7 mm
- net SWCLK: track 0.00 -> 20.0 mm, vias 0 -> 2
- net SWDIO: track 0.00 -> 14.8 mm, vias 0 -> 1
- net Button: track 0.00 -> 14.0 mm, vias 0 -> 1
- net GND: track 0.00 -> 5.37 mm, vias 0 -> 3
- net LED_DIN: track 0.00 -> 5.34 mm
- added copper zone on B.Cu, net GND
- added copper zone on F.Cu, net GND
Other:
- board outline added: 27 x 27 mm
- board text added: "LJB"
