File: PCBs/FinalProjPCB/FinalProjPCB.kicad_pcb (KiCad board)
At the start: 2 copper layers, 87.2 x 109.2 mm, 20 parts, among them J1 Conn_01x20, J2 Conn_01x05, J3 Conn_01x20, SW7 SW_SPDT, U1 XMSM0G3507SDGS28R

Commit message: updated pcb
Connections:
- J3 pad 1: (no net) -> unconnected-(J3-Pin_1-Pad1)
- U1 pad 17: unconnected-(U1-PA14/CLK_OUT/A0_12-Pad17) -> SD_CS
- U1 pad 18: SD_CS -> unconnected-(U1-PA15/A1_0-Pad18)
- U1 pad 25: BUTTON_UP_IO -> BUZZER_IO
- U1 pad 26: BUTTON_RIGHT_IO -> BUTTON_UP_IO
- U1 pad 27: BUTTON_LEFT_IO -> BUTTON_RIGHT_IO
- U1 pad 28: BUZZER_IO -> BUTTON_LEFT_IO
Routing:
- net BUZZER_IO: track 35.6 -> 32.9 mm
- net BUTTON_LEFT_IO: track 60.8 -> 59.7 mm
- net SD_CS: track 21.0 -> 20.0 mm
