File: PCBs/FinalProjPCB/FinalProjPCB.kicad_sch (KiCad schematic)
At the start: 0 parts

Commit message: final proj pcb v1
Parts:
- added A1, B1, DOWN1, LEFT1, RIGHT1, UP1: SW_SPST, Button_Switch_SMD:SW_SPST_PTS647_Sx38, symbol Switch:SW_SPST
- added BT1: Battery_Cell, Battery:BatteryHolder_Keystone_1060_1x2032, symbol Device:Battery_Cell
- added BZ1: Buzzer, Buzzer_Beeper:Buzzer_Murata_PKLCS1212E, symbol Device:Buzzer
- added C1: 10uF, Capacitor_SMD:C_0603_1608Metric, symbol Device:C
- added C2: 0.1uF, Capacitor_SMD:C_0603_1608Metric_Pad1.08x0.95mm_HandSolder, symbol Device:C
- added C3: 100uF, Capacitor_SMD:C_1206_3216Metric, symbol Device:C
- added C4: 0.47 uF, Capacitor_SMD:C_0805_2012Metric, symbol Device:C
- added C6: 10nF, Capacitor_SMD:C_0402_1005Metric, symbol Device:C
- added J1, J3: Conn_01x20, Connector_PinHeader_2.54mm:PinHeader_1x20_P2.54mm_Vertical, symbol Connector_Generic:Conn_01x20
- added J2: Conn_01x05, Connector_PinHeader_2.54mm:PinHeader_1x05_P2.54mm_Horizontal, symbol Connector_Generic:Conn_01x05
- added R5: 47k, Resistor_SMD:R_0603_1608Metric, symbol Device:R_US
- added R6: 100k, Resistor_SMD:R_0402_1005Metric, symbol Device:R_US
- added SW7: SW_SPDT, ELEC327-Kicad:SW_EG1270, symbol Switch:SW_SPDT
- added U1: XMSM0G3507SDGS28R, VSSOP28_DGS_TEX, symbol MSPM0G3507:XMSM0G3507SDGS28R
Connections:
- new net: BT1.1 (+), SW7.2 (B)
- new net BUTTON_A_IO: A1.1 (A), U1.21 (PA18/A1_3)
- new net BUTTON_B_IO: B1.1 (A), U1.20 (PA17/A1_2)
- new net BUTTON_DOWN_IO: DOWN1.1 (A), U1.24 (PA21/A1_7/VREF-)
- new net BUTTON_LEFT_IO: LEFT1.1 (A), U1.27 (PA24/A0_3)
- new net BUTTON_RIGHT_IO: RIGHT1.1 (A), U1.26 (PA23/VREF+)
- new net BUTTON_UP_IO: U1.25 (PA22/CLK_OUT/A0_7), UP1.1 (A)
- new net BUZZER_IO: BZ1.1 (+), U1.28 (PA25/A0_2)
- new net GND: A1.2 (B), B1.2 (B), BT1.2 (-), BZ1.2 (-), C1.2, C2.2, C3.2, C4.2, C6.2, DOWN1.2 (B), J1.1 (Pin_1), J2.1 (Pin_1), LEFT1.2 (B), R6.1, RIGHT1.2 (B), U1.8 (VSS), UP1.2 (B)
- new net NRST: C6.1, J2.3 (Pin_3), R5.1, U1.6 (NRST)
- new net ROSC: R6.2, U1.9 (PA2_/_ROSC)
- new net SD_CS: J1.19 (Pin_19), U1.18 (PA15/A1_0)
- new net SD_DET: J1.20 (Pin_20), U1.19 (PA16/A1_1/FCC_IN)
- new net SPI_CLK: J1.4 (Pin_4), U1.13 (PA6/HFCLK_IN/HFXOUT)
- new net SPI_CS: J1.7 (Pin_7), U1.10 (PA3_/_LFXIN)
- new net SPI_DC: J1.8 (Pin_8), U1.1 (PA26/A0_1)
- new net SPI_PICO: J1.6 (Pin_6), U1.12 (PA5/HFXIN/FCC_IN)
- new net SPI_POCI: J1.5 (Pin_5), U1.11 (PA4_/_LFCLK_IN_/_LFXOUT)
- new net SPI_RST: J1.9 (Pin_9), U1.2 (PA27/RTC_OUT/A0_0)
- new net SWCLK: J2.5 (Pin_5), U1.23 (PA20/SWCLK)
- new net SWDIO: J2.4 (Pin_4), U1.22 (PA19/SWDIO)
- new net VCORE: C4.1, U1.3 (VCORE)
- new net VDD: C1.1, C2.1, C3.1, J1.2 (Pin_2), J2.2 (Pin_2), R5.2, SW7.1 (A), U1.7 (VDD)
- no-connect marks 0 -> 20
Other:
- note added: "Debug Iface"
- note added: "Reset Circuit (RC delay enables programming)"
- note added: "SYSOSC Freq Loop Stabilization (100 kOhm 1% tol, 25 ppm/C)"
- note added: "Tank Capacitor (Should be placed close to device)"

Commit message: updated pcb
Connections:
- net BUTTON_LEFT_IO: now also U1.28 (PA25/A0_2); no longer U1.27 (PA24/A0_3)
- net BUTTON_RIGHT_IO: now also U1.27 (PA24/A0_3); no longer U1.26 (PA23/VREF+)
- net BUTTON_UP_IO: now also U1.26 (PA23/VREF+); no longer U1.25 (PA22/CLK_OUT/A0_7)
- net BUZZER_IO: now also U1.25 (PA22/CLK_OUT/A0_7); no longer U1.28 (PA25/A0_2)
- net SD_CS: now also U1.17 (PA14/CLK_OUT/A0_12); no longer U1.18 (PA15/A1_0)
